File: HW2/PIC32/PIC32.brd (EAGLE design)
At the start: 50 x 50 mm, 23 parts, among them J4 AMP FCI 10103594-0001LF

Commit message: working spi channel
Parts:
- moved J2 107.0 mm to (-52.1, 52.1), turned to 0 degrees
- moved C1 88.1 mm to (-45.7, 31.8), turned to 0 degrees
- moved U$2 86.4 mm to (-49.5, 40.6), turned to 0 degrees
- moved J4 83.6 mm to (-34.3, 22.9), turned to 0 degrees
- moved C4 79.0 mm to (-50.8, 31.8), turned to 0 degrees
- moved MPLAB_SNAP 71.9 mm to (-47.0, 57.1), turned to 0 degrees
- moved C5 71.3 mm to (-52.1, 21.6), turned to 0 degrees
- moved R4 71.2 mm to (-48.3, 47.0), turned to 0 degrees
- moved C2 67.4 mm to (-41.9, 39.4)
- moved USER_PUSH 65.9 mm to (-40.6, 33.0), turned to 0 degrees
- moved U$3 63.7 mm to (-31.8, 33.0)
- moved U$1 59.9 mm to (-30.5, 3.81)
- moved GREEN 58.0 mm to (-21.6, 53.3), turned to 0 degrees
- moved U$4 57.6 mm to (-35.6, 39.4), turned to 0 degrees
- moved R1 56.7 mm to (-38.1, 47.0), turned to 0 degrees
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Connections:
- net N$7 renamed B0
- net N$9 renamed B1
- removed net 5V_USB: C4.1, U$4.VIN, U$5.3
- removed net N$5: U$1.19
- removed net N$6: U$1.20
- new net 5V: C4.1, J3.7, U$4.VIN, U$5.3
- new net A0: J2.1, U$1.19
- new net A1: J2.2, U$1.20
- new net A10: U$1.12
- new net A4: J2.6
- new net A7: U$1.13
- new net A8: U$1.32
- new net A9: U$1.35
- new net B13: J3.3, U$1.11
- new net B14: J3.2, U$1.14
- new net B15: J3.1, U$1.15
- new net B2: J2.3, U$1.23
- new net B3: J2.4, U$1.24
- new net B4: J2.5
- new net B5: U$1.41
- new net B7: J3.6, U$1.43
- new net B8: J3.5, U$1.44
- new net B9: J3.4, U$1.1
- new net C0: U$1.25
- new net C1: U$1.26
- new net C3: U$1.36
- new net C4: U$1.37
- new net C5: U$1.38
- new net C6: U$1.2
- new net C7: U$1.3
- new net C8: U$1.4
- new net C9: U$1.5
- new net N$26: U$1.27
- new net VBUS: U$1.42
- net +3V3: no longer MPLAB_SNAP.4
- net 3.3V: now also J2.7
- net GND: now also J2.8, J3.8; no longer MPLAB_SNAP.3
Routing:
- net N$11: track 4.57 -> 0.00 mm
- removed copper zone on layer 16, net GND
Other:
- board size 50 x 50 mm -> 410 x 250 mm

Commit message: CAD images of wheel and box
Parts:
- moved MPLAB_SNAP 111.0 mm to (47.9, -0.49), turned to 90 degrees
- moved J2 107.3 mm to (-9.57, -46.4)
- moved R4 107.1 mm to (40.8, -12.5), turned to 180 degrees
- moved C1 87.8 mm to (33.2, -6.72), turned to 90 degrees
- moved C5 85.1 mm to (32.9, 26.6)
- moved C4 84.6 mm to (33.7, 35.2)
- moved J4 81.0 mm to (43.3, 46.1), turned to 180 degrees
- moved U$2 79.2 mm to (19.4, 1.47), turned to 90 degrees
- moved U$4 78.1 mm to (42.4, 34.1), turned to 270 degrees
- moved RED 77.9 mm to (41.7, 24.0), turned to 90 degrees
- moved R3 71.6 mm to (37.9, 19.0), turned to 180 degrees
- moved J3 66.5 mm to (-46.1, -8.02), turned to 90 degrees
- moved USER_PUSH 63.3 mm to (21.6, 44.5), turned to 180 degrees
- moved C6 56.9 mm to (-0.74, -13.1)
- moved R1 56.6 mm to (16.5, 32.1), turned to 270 degrees
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Connections:
- removed net N$1: USER_PUSH.1
- removed net N$2: GREEN.A
- net +3V3: no longer C1.1, C6.1, U$1.17, U$1.28
- net 3.3V: now also C1.1, C6.1, MPLAB_SNAP.4, U$1.17, U$1.28
- net GND: now also MPLAB_SNAP.3
- net GREEN_LED: now also GREEN.A
- net USER_PUSH: now also USER_PUSH.1
Other:
- board size 410 x 250 mm -> 100 x 100 mm

Commit message: HW15
Parts:
- moved R4 30.5 mm to (47.5, 17.2), turned to 90 degrees
- moved C1 10.9 mm to (30.2, 3.72), turned to 270 degrees
- moved C6 2.05 mm to (-2.76, -13.4), turned to 180 degrees
- moved C7 0.40 mm to (-16.8, -8.59), turned to 0 degrees
- turned C2 to 180 degrees
Connections:
- removed net +3V3: R4.2
- net 3.3V: now also R4.2
Routing:
- net 3.3V: track 0.00 -> 206.3 mm, vias 0 -> 6
- net 5V: track 0.00 -> 121.0 mm
- net N_MCLR: track 0.00 -> 95.1 mm, vias 0 -> 2
- net PGED: track 0.00 -> 55.6 mm, vias 0 -> 2
- net PGEC: track 0.00 -> 54.8 mm, vias 0 -> 2
- net USER_PUSH: track 0.00 -> 52.2 mm
- net B7: track 0.00 -> 50.7 mm
- net B15: track 0.00 -> 50.1 mm
- net B3: track 0.00 -> 48.3 mm
- net B2: track 0.00 -> 46.7 mm
- net B14: track 0.00 -> 45.3 mm
- net A0: track 0.00 -> 45.1 mm
- net A1: track 0.00 -> 44.4 mm
- net B8: track 0.00 -> 43.6 mm
- net GREEN_LED: track 0.00 -> 43.1 mm
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- added copper zone on layer 16, net GND
